Commit message: fix moveit config

File: sawyer_description/urdf/full_sawyer.urdf.xacro (robot description, xacro)
@@ -690,3 +690,107 @@
     <dynamics damping="100.0" friction="500.0"/>
   </joint>
+   <!-- ros2 control tag -->
+    <ros2_control name="robot_6_dof" type="system">
+      <hardware>
+        <plugin>sawyer_robot_driver/RobotSystem</plugin>
+      </hardware>
+      <joint name="right_j0">
+        <command_interface name="position">
+          <param name="min">{-2*pi}</param>
+          <param name="max">{2*pi}</param>
+        </command_interface>
+        <command_interface name="velocity">
+          <param name="min">-3.15</param>
+          <param name="max">3.15</param>
+        </command_interface>
+        <state_interface name="position">
+          <param name="initial_value">0.0</param>
+        </state_interface>
+        <state_interface name="velocity"/>
+      </joint>
+      <joint name="right_j1">
+        <command_interface name="position">
+          <param name="min">{-2*pi}</param>
+          <param name="max">{2*pi}</param>
+        </command_interface>
+        <command_interface name="velocity">
+          <param name="min">-3.15</param>
+          <param name="max">3.15</param>
+        </command_interface>
+        <state_interface name="position">
+          <param name="initial_value">0.0</param>
+        </state_interface>
+        <state_interface name="velocity"/>
+      </joint>
+      <joint name="right_j2">
+        <command_interface name="position">
+          <param name="min">{-pi}</param>
+          <param name="max">{pi}</param>
+        </command_interface>
+        <command_interface name="velocity">
+          <param name="min">-3.15</param>
+          <param name="max">3.15</param>
+        </command_interface>
+        <state_interface name="position">
+          <param name="initial_value">0.0</param>
+        </state_interface>
+        <state_interface name="velocity"/>
+      </joint>
+      <joint name="right_j3">
+        <command_interface name="position">
+          <param name="min">{-2*pi}</param>
+          <param name="max">{2*pi}</param>
+        </command_interface>
+        <command_interface name="velocity">
+          <param name="min">-3.2</param>
+          <param name="max">3.2</param>
+        </command_interface>
+        <state_interface name="position">
+          <param name="initial_value">0.0</param>
+        </state_interface>
+        <state_interface name="velocity"/>
+      </joint>
+      <joint name="right_j4">
+        <command_interface name="position">
+          <param name="min">{-2*pi}</param>
+          <param name="max">{2*pi}</param>
+        </command_interface>
+        <command_interface name="velocity">
+          <param name="min">-3.2</param>
+          <param name="max">3.2</param>
+        </command_interface>
+        <state_interface name="position">
+          <param name="initial_value">0.0</param>
+        </state_interface>
+        <state_interface name="velocity"/>
+      </joint>
+      <joint name="right_j5">
+        <command_interface name="position">
+          <param name="min">{-2*pi}</param>
+          <param name="max">{2*pi}</param>
+        </command_interface>
+        <command_interface name="velocity">
+          <param name="min">-3.2</param>
+          <param name="max">3.2</param>
+        </command_interface>
+        <state_interface name="position">
+          <param name="initial_value">0.0</param>
+        </state_interface>
+        <state_interface name="velocity"/>
+      </joint>
+      <joint name="right_j6">
+        <command_interface name="position">
+          <param name="min">{-2*pi}</param>
+          <param name="max">{2*pi}</param>
+        </command_interface>
+        <command_interface name="velocity">
+          <param name="min">-3.2</param>
+          <param name="max">3.2</param>
+        </command_interface>
+        <state_interface name="position">
+          <param name="initial_value">0.0</param>
+        </state_interface>
+        <state_interface name="velocity"/>
+      </joint>
+    </ros2_control>
 </robot>

Commit message: add moveit config and ros2 control

File: sawyer_description/urdf/full_sawyer.urdf.xacro (robot description, xacro)
@@ -143,5 +143,5 @@
     <child link="right_l0"/>
     <axis xyz="0 0 1"/>
-    <limit effort="80.0" lower="-3.0503" upper="3.0503" velocity="1.74"/>
+    <limit effort="80.0" lower="-1000" upper="1000" velocity="1.74"/>
   </joint>
   <link name="head">
@@ -170,5 +170,5 @@
     <child link="head"/>
     <axis xyz="0 0 1"/>
-    <limit effort="8" lower="-5.0952" upper="0.9064" velocity="1.8"/>
+    <limit effort="8" lower="-1000" upper="1000" velocity="1.8"/>
   </joint>
   <link name="right_torso_itb">
@@ -210,5 +210,5 @@
     <child link="right_l1"/>
     <axis xyz="0 0 1"/>
-    <limit effort="80.0" lower="-3.8095" upper="2.2736" velocity="1.328"/>
+    <limit effort="80.0" lower="-1000" upper="1000" velocity="1.328"/>
   </joint>
   <link name="right_l2">
@@ -237,5 +237,5 @@
     <child link="right_l2"/>
     <axis xyz="0 0 1"/>
-    <limit effort="40.0" lower="-3.0426" upper="3.0426" velocity="1.957"/>
+    <limit effort="40.0" lower="-1000" upper="1000" velocity="1.957"/>
   </joint>
   <link name="right_l3">
@@ -264,5 +264,5 @@
     <child link="right_l3"/>
     <axis xyz="0 0 1"/>
-    <limit effort="40.0" lower="-3.0439" upper="3.0439" velocity="1.957"/>
+    <limit effort="40.0" lower="-1000" upper="1000" velocity="1.957"/>
   </joint>
   <link name="right_l4">
@@ -291,5 +291,5 @@
     <child link="right_l4"/>
     <axis xyz="0 0 1"/>
-    <limit effort="9.0" lower="-2.9761" upper="2.9761" velocity="3.485"/>
+    <limit effort="9.0" lower="-1000" upper="1000" velocity="3.485"/>
   </joint>
   <link name="right_arm_itb">
@@ -331,5 +331,5 @@
     <child link="right_l5"/>
     <axis xyz="0 0 1"/>
-    <limit effort="9.0" lower="-2.9761" upper="2.9761" velocity="3.485"/>
+    <limit effort="9.0" lower="-1000" upper="1000" velocity="3.485"/>
   </joint>
   <link name="right_hand_camera"/>
@@ -372,5 +372,5 @@
     <child link="right_l6"/>
     <axis xyz="0 0 1"/>
-    <limit effort="9.0" lower="-4.7124" upper="4.7124" velocity="4.545"/>
+    <limit effort="9.0" lower="-1000" upper="1000" velocity="4.545"/>
   </joint>
   <link name="right_hand">
@@ -678,5 +678,5 @@
     <parent link="right_electric_gripper_base"/>
     <child link="right_gripper_l_finger"/>
-    <limit effort="20.0" lower="0.0" upper="0.020833" velocity="5.0"/>
+    <limit effort="20.0" lower="-1000" upper="1000" velocity="5.0"/>
     <dynamics damping="100.0" friction="500.0"/>
   </joint>
@@ -686,5 +686,5 @@
     <parent link="right_electric_gripper_base"/>
     <child link="right_gripper_r_finger"/>
-    <limit effort="20.0" lower="-0.020833" upper="0.0" velocity="5.0"/>
+    <limit effort="20.0" lower="-1000" upper="1000" velocity="5.0"/>
     <mimic joint="right_gripper_l_finger_joint" multiplier="-1.0"/>
     <dynamics damping="100.0" friction="500.0"/>
@@ -696,8 +696,4 @@
       </hardware>
       <joint name="right_j0">
-        <command_interface name="position">
-          <param name="min">{-2*pi}</param>
-          <param name="max">{2*pi}</param>
-        </command_interface>
         <command_interface name="velocity">
           <param name="min">-3.15</param>
@@ -711,8 +707,4 @@
       </joint>
       <joint name="right_j1">
-        <command_interface name="position">
-          <param name="min">{-2*pi}</param>
-          <param name="max">{2*pi}</param>
-        </command_interface>
         <command_interface name="velocity">
           <param name="min">-3.15</param>
@@ -726,8 +718,4 @@
       </joint>
       <joint name="right_j2">
-        <command_interface name="position">
-          <param name="min">{-pi}</param>
-          <param name="max">{pi}</param>
-        </command_interface>
         <command_interface name="velocity">
           <param name="min">-3.15</param>
@@ -741,8 +729,4 @@
       </joint>
       <joint name="right_j3">
-        <command_interface name="position">
-          <param name="min">{-2*pi}</param>
-          <param name="max">{2*pi}</param>
-        </command_interface>
         <command_interface name="velocity">
           <param name="min">-3.2</param>
@@ -756,8 +740,4 @@
       </joint>
       <joint name="right_j4">
-        <command_interface name="position">
-          <param name="min">{-2*pi}</param>
-          <param name="max">{2*pi}</param>
-        </command_interface>
         <command_interface name="velocity">
           <param name="min">-3.2</param>
@@ -771,8 +751,4 @@
       </joint>
       <joint name="right_j5">
-        <command_interface name="position">
-          <param name="min">{-2*pi}</param>
-          <param name="max">{2*pi}</param>
-        </command_interface>
         <command_interface name="velocity">
           <param name="min">-3.2</param>
@@ -786,8 +762,4 @@
       </joint>
       <joint name="right_j6">
-        <command_interface name="position">
-          <param name="min">{-2*pi}</param>
-          <param name="max">{2*pi}</param>
-        </command_interface>
         <command_interface name="velocity">
           <param name="min">-3.2</param>
