Commit message: add teleop and robot_library pybind

File: teleop_script/sawyer.urdf (robot description, URDF)
Before this commit: robot sawyer, 21 links, 20 joints
Links:
- added link camera_base_link
- added link camera_bottom_screw_frame
- added link camera_link, mass 0.072; collision box size=0.02505 0.09 0.025; visual mesh filename=package://realsense2_description/meshes/d435.dae
- added link controller_box; collision box size=0.22 0.4 0.53
- added link pedestal, mass 60.86397744; collision cylinder length=0.62 radius=0.18; visual mesh filename=package://custom_sawyer_description/meshes/sawyer_pv/pedest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
- added link pedestal_feet; collision box size=0.77 0.7 0.31
- added link right_connector_plate_base, mass 0.0; collision cylinder length=0.0302 radius=0.04; visual mesh filename=package://intera_tools_description/meshes/connector_plate/c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
- added link right_connector_plate_mount
- added link right_electric_gripper_base, mass 2e-06; collision cylinder length=0.1 radius=0.029; visual mesh filename=package://intera_tools_description/meshes/electric_gripper/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
- added link right_gripper_base, mass 0.47
- added link right_gripper_l_finger, mass 0.001; collision box size=0.01 0.0135 0.075; collision box size=0.01 0.05 0.017
- added link right_gripper_l_finger_tip, mass 0.001; collision box size=0.016 0.007 0.037; visual mesh filename=package://intera_tools_description/meshes/electric_gripper/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
- added link right_gripper_r_finger, mass 0.001; collision box size=0.01 0.0135 0.075; collision box size=0.01 0.05 0.017
- added link right_gripper_r_finger_tip, mass 0.001; collision box size=0.016 0.007 0.037; visual mesh filename=package://intera_tools_description/meshes/electric_gripper/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
- added link right_gripper_tip, mass 2e-06
- link head: geometry collision sphere radius=0.18; visual mesh filename=package://custom_sawyer_description/meshes/sawyer_pv/head.D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
- link right_arm_base_link: geometry collision cylinder length=0.24 radius=0.08; visual mesh filename=package://custom_sawyer_description/meshes/sawyer_pv/base.D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
- link right_arm_itb: mass None -> 0.0001
- link right_hand: mass None -> 1.0E-08
- link right_hand_camera: mass None -> 0.0
- link right_l0: geometry collision sphere radius=0.07; visual mesh filename=package://custom_sawyer_description/meshes/sawyer_mp3/l0.DAE
- link right_l1: geometry collision sphere radius=0.07; visual mesh filename=package://custom_sawyer_description/meshes/sawyer_mp3/l1.DAE
- link right_l1_2: mass None -> 1.0E-08
- link right_l2: geometry collision cylinder length=0.34 radius=0.06; visual mesh filename=package://custom_sawyer_description/meshes/sawyer_pv/l2.DAE
- link right_l2_2: mass None -> 1.0E-08
- link right_l3: geometry collision sphere radius=0.06; visual mesh filename=package://custom_sawyer_description/meshes/sawyer_pv/l3.DAE
- link right_l4: geometry collision cylinder length=0.30 radius=0.045; visual mesh filename=package://custom_sawyer_description/meshes/sawyer_pv/l4.DAE
- link right_l4_2: mass None -> 1.0E-08
- link right_l5: geometry collision sphere radius=0.06; visual mesh filename=package://custom_sawyer_description/meshes/sawyer_pv/l5.DAE
- link right_l6: geometry collision cylinder length=0.05 radius=0.055; visual mesh filename=package://custom_sawyer_description/meshes/sawyer_mp1/l6.DAE
- link right_torso_itb: mass None -> 0.0001
- link screen: mass None -> 0.0001
- link torso: mass None -> 0.0001
Joints:
- added joint camera_joint: type fixed, parent camera_base_link, child camera_bottom_screw_frame, origin xyz=0 0 0 rpy=0 0 0
- added joint camera_link_joint: type fixed, parent camera_bottom_screw_frame, child camera_link, origin xyz=0.010600000000000002 0.0175 0.0125 rpy=0 0 0
- added joint controller_box_fixed: type fixed, parent base, child controller_box, origin xyz=0.0 0.0 0.0 rpy=0 0 0
- added joint pedestal_feet_fixed: type fixed, parent base, child pedestal_feet, origin xyz=0.0 0.0 0.0 rpy=0 0 0
- added joint pedestal_fixed: type fixed, parent base, child pedestal, origin xyz=0.0 0.0 0.0 rpy=0 0 0
- added joint right_connector_plate_base_joint: type fixed, parent right_gripper_base, child right_connector_plate_base, origin xyz=0 0 0.0018 rpy=0 0 0
- added joint right_connector_plate_mount_joint: type fixed, parent right_connector_plate_base, child right_connector_plate_mount, origin xyz=0 0 0.0176 rpy=0 0 0
- added joint right_electric_gripper_base_joint: type fixed, parent right_connector_plate_mount, child right_electric_gripper_base, origin xyz=0 0 0 rpy=0 0 0
- added joint right_gripper_base_joint: type fixed, parent right_hand, child right_gripper_base, origin xyz=0 0 -0.005 rpy=0 0 0
- added joint right_gripper_l_finger_joint: type prismatic, parent right_electric_gripper_base, child right_gripper_l_finger, origin xyz=0.003 -0.0014999999999999996 0.04552 rpy=0 0 0, axis 0 1 0, limit lower=0.0 upper=0.020833 effort=20.0 velocity=5.0
- added joint right_gripper_l_finger_tip_joint: type fixed, parent right_gripper_l_finger, child right_gripper_l_finger_tip, origin xyz=0.0 0.01725 0.075 rpy=0 0 0
- added joint right_gripper_r_finger_joint: type prismatic, parent right_electric_gripper_base, child right_gripper_r_finger, origin xyz=0.003 0.0014999999999999996 0.04552 rpy=0 0 0, axis 0 1 0, limit lower=-0.020833 upper=0.0 effort=20.0 velocity=5.0, mimic joint=right_gripper_l_finger_joint multiplier=-1.0
- added joint right_gripper_r_finger_tip_joint: type fixed, parent right_gripper_r_finger, child right_gripper_r_finger_tip, origin xyz=0.0 -0.01725 0.075 rpy=0 0 0
- added joint right_gripper_tip_joint: type fixed, parent right_gripper_base, child right_gripper_tip, origin xyz=0 0 0.14062 rpy=0 0 0
- added joint right_l6_to_camera: type fixed, parent right_l6, child camera_base_link, origin xyz=0 0.038279 0.028525 rpy=-1.57079632679 4.71238898 0, axis 0 0 0
- joint right_j6: limit (none) -> lower=-4.7124 upper=4.7124 effort=9.0 velocity=4.545
