Commit message: fixed the bugs blocking this from building into urdf

File: intera_tools_description/urdf/dental_drill/dental_drill.xacro (robot description, xacro)
@@ -1,5 +1,5 @@
 <?xml version="1.0" encoding="utf-8"?>
 <robot xmlns:xacro="https://ros.org/wiki/xacro" name="dental_drill">
-  <xacro:macro name="dental_drill" params="prefix connected_to">
+  <xacro:macro name="dental_drill" params="prefix">
     <link name="${prefix}dental_drill_joint" type="fixed">
       <inertial>

File: sawyer_description/urdf/sawyer.urdf.xacro (robot description, xacro)
@@ -7,10 +7,10 @@
   <xacro:arg name="electric_gripper" default="false"/>
   <!-- Sawyer Base URDF -->
-  <xacro:include filename="package://sawyer_description/urdf/sawyer_base.urdf.xacro">
+  <xacro:include filename="$(find sawyer_description)/urdf/sawyer_base.urdf.xacro">
     <xacro:arg name="gazebo" value="${gazebo}"/>
     <xacro:arg name="pedestal" value="${pedestal}"/>
   </xacro:include>
   <xacro:if value="$(arg gazebo)">
-  <xacro:include filename="package://sawyer_description/urdf/sawyer_base.gazebo.xacro">
+  <xacro:include filename="$(find sawyer_description)/urdf/sawyer_base.gazebo.xacro">
     <xacro:arg name="static" value="${static}"/>
     <xacro:arg name="pedestal" value="${pedestal}"/>
@@ -19,5 +19,5 @@
   <!-- Electric Gripper End Effector -->
   <xacro:if value="$(arg electric_gripper)">
-  <xacro:include filename="package://sawyer_description/urdf/sawyer_electric_gripper.urdf.xacro">
+  <xacro:include filename="$(find sawyer_description)/urdf/sawyer_electric_gripper.urdf.xacro">
     <xacro:arg name="gazebo" value="${gazebo}"/>
   </xacro:include>
@@ -25,5 +25,5 @@
   <!-- Dental Drill End Effector -->
   <xacro:if value="$(arg dental_drill)">
-  <xacro:include filename="package://sawyer_description/urdf/sawyer_dental_drill.urdf.xacro">
+  <xacro:include filename="$(find sawyer_description)/urdf/sawyer_dental_drill.urdf.xacro">
     <xacro:arg name="gazebo" value="${gazebo}"/>
   </xacro:include>

Commit message: fixed bugs - not the full robot displays correctly including the dental drill

File: intera_tools_description/urdf/dental_drill/dental_drill.xacro (robot description, xacro)
@@ -2,5 +2,5 @@
 <robot xmlns:xacro="https://ros.org/wiki/xacro" name="dental_drill">
   <xacro:macro name="dental_drill" params="prefix">
-    <link name="${prefix}dental_drill_joint" type="fixed">
+    <link name="${prefix}_dental_drill_tip" type="fixed">
       <inertial>
         <origin rpy="0 0 0" xyz="0 0 0"/>
@@ -26,18 +26,13 @@
       </inertial>
     </link>
-    <joint name="${prefix}_gripper_base" type="fixed">
+    <joint name="${prefix}_endpoint" type="fixed">
       <origin rpy="0 0 0" xyz="0 0 0"/>
       <parent link="${prefix}_hand"/>
-      <child link="${prefix}_gripper_base"/>
-    </joint>
-    <joint name="${prefix}_endpoint" type="fixed">
-      <origin rpy="0 0 0" xyz="0 0 0"/>
-      <parent link="${prefix}_gripper_base"/>
-      <child link="${prefix}_gripper"/>
+      <child link="${prefix}_dental_drill"/>
     </joint>
     <joint name="${prefix}tip_frame" type="fixed">
       <origin rpy="0 0 0" xyz="0 -0.01744 0.149"/>
-      <parent link="${prefix}_gripper_base"/>
-      <child link="${prefix}_dental_drill"/>
+      <parent link="${prefix}_dental_drill"/>
+      <child link="${prefix}_dental_drill_tip"/>
     </joint>
   </xacro:macro>

Commit message: adjusted mount position of the drill and also added the drill tip

File: intera_tools_description/urdf/dental_drill/dental_drill.xacro (robot description, xacro)
@@ -3,4 +3,10 @@
   <xacro:macro name="dental_drill" params="prefix">
     <link name="${prefix}_dental_drill_tip" type="fixed">
+      <visual>
+        <origin rpy="${pi/2} 0 0" xyz="0 0.00372 0"/>
+        <geometry>
+          <cylinder length="0.00744" radius="0.001"/>
+        </geometry>
+      </visual>
       <inertial>
         <origin rpy="0 0 0" xyz="0 0 0"/>
@@ -27,5 +33,5 @@
     </link>
     <joint name="${prefix}_endpoint" type="fixed">
-      <origin rpy="0 0 0" xyz="0 0 0"/>
+      <origin rpy="0 0 0" xyz="0 -0.028 0"/>
       <parent link="${prefix}_hand"/>
       <child link="${prefix}_dental_drill"/>

Commit message: added collition detection for the drill tip

File: intera_tools_description/urdf/dental_drill/dental_drill.xacro (robot description, xacro)
@@ -9,4 +9,10 @@
         </geometry>
       </visual>
+      <collision>
+        <origin rpy="${pi/2} 0 0" xyz="0 0.00372 0"/>
+        <geometry>
+          <cylinder length="0.00744" radius="0.001"/>
+        </geometry>
+      </collision>
       <inertial>
         <origin rpy="0 0 0" xyz="0 0 0"/>
